File: Hardware/Kicad/ESP32CAM Shield.kicad_pcb (KiCad board)
At the start: 4 copper layers, 29 x 45 mm, 47 parts, among them J1 Conn_01x08_Socket, J2 Conn_01x08_Socket, J3 JST-PH, J4 USB_C_Receptacle_USB2.0_14P, Q1 AO3401A, Q2 FS8205A, SW1 SW_SPDT, SW2 SW_SPDT, U1 MCP73831-2-OT, U2 AP2112K-3.3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

Commit message: Added BOOT and ON/OFF switches text
Other:
- board text added: "BOOT"
- board text added: "ON/OFF"
Changed lines of the file:
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@@
 		(descr "Ultraminiature Surface Mount Slide Switch, right-angle, https://www.ckswitches.com/media/1424/pcm.pdf")
 		(property "Reference" "SW2"
-			(at 4.92 0.33 180)
+			(at -4.986 0.33 180)
 			(layer "F.SilkS")
 			(effects
@@
 		)
 		(fp_text user "${REFERENCE}"
-			(at 4.92 0.33 180)
+			(at -4.986 0.33 180)
 			(layer "F.Fab")
 			(effects
@@
 		(descr "Ultraminiature Surface Mount Slide Switch, right-angle, https://www.ckswitches.com/media/1424/pcm.pdf")
 		(property "Reference" "SW1"
-			(at -5.394 0.33 180)
+			(at 5.147 0.33 180)
 			(layer "F.SilkS")
 			(effects
@@
 		)
 		(fp_text user "${REFERENCE}"
-			(at -5.394 0.33 180)
+			(at 5.147 0.33 180)
 			(layer "F.Fab")
 			(effects
@@
 		(layer "Edge.Cuts")
 	)
+	(gr_text "ON/OFF"
+		(at 124.841 98.044 0)
+		(layer "F.SilkS")
+		(effects
+			(font
+				(size 1 1)
+				(thickness 0.1)
+			)
+			(justify left bottom)
+		)
+	)
+	(gr_text "BOOT"
+		(at 149.225 98.425 0)
+		(layer "F.SilkS")
+		(effects
+			(font
+				(size 1 1)
+				(thickness 0.1)
+			)
+			(justify left bottom)
+		)
+	)
 	(gr_text "Designed by VonMartins \nRev 1.0 - 10/05/2025"
